File: KiCad/riscv-phone/riscv-phone.kicad_pcb (KiCad board)
At the start: 2 copper layers, 46.4 x 52.8 mm, 93 parts, among them J1 USB_B_Micro, J2 Conn_01x04, J3 Conn_01x04, J4 Conn_01x11, J5 Conn_01x10, J7 Conn_01x02, Q1 Q_DUAL_NMOS_S1G1D2S2G2D1, Q2 IRLML6402, U1 FE310-G000, U12 SC18IS600, U17 74AHC1G08, U18 M95256-WMN6P, U2 IL25LP128, U5 74CBTLV3257, U9 FT2232H, U90 TLV75533PDBV, U91 TLV75518PDBV, X1 SiT1533, Y1 16 MHz, Y2 12 MHz

Commit message: Revision 2.0
Parts:
- removed the C11 at (128.8, 141.2)
- removed the C12 at (144.1, 139.3)
- removed the C13 at (139.1, 151.6)
- removed the C14 at (135.6, 136.4)
- removed the C17 at (132.8, 146.3)
- removed the C18 at (126.7, 143.8)
- removed C59, C60: 0.1uF, Capacitor_SMD:C_0603_1608Metric
- removed the C7 at (127.0, 132.8)
- removed the C9 at (140.7, 131.7)
- removed D1: 1N4448W, Diode_SMD:D_SOD-123
- removed D3: BAT54L, Package_TO_SOT_SMD:SOT-23
- removed the G*** at (154.2, 113.8)
- removed the J2 at (119.9, 153.4)
- removed Q1: Q_DUAL_NMOS_S1G1D2S2G2D1, Package_TO_SOT_SMD:SOT-363_SC-70-6
- removed Q2: IRLML6402, Package_TO_SOT_SMD:SOT-23
- removed the R11 at (124.2, 151.8)
- removed R27, R28, R30: 1k, Resistor_SMD:R_0603_1608Metric
- removed R34, R35: 2.2k, Resistor_SMD:R_0603_1608Metric
- removed R53: 100k, Resistor_SMD:R_0603_1608Metric
- removed R54: 4.7k, Resistor_SMD:R_0603_1608Metric
- removed the R6 at (121.9, 135.4)
- removed the R9 at (123.7, 146.6)
- removed TP1: TestPoint, TestPoint:TestPoint_Pad_2.0x2.0mm
- removed U12: SC18IS600, Package_SO:TSSOP-16_4.4x5mm_P0.65mm
- removed U17: 74AHC1G08, Package_TO_SOT_SMD:SOT-23-5
- removed U18: M95256-WMN6P, Package_SO:SOIC-8_3.9x4.9mm_P1.27mm
- removed the U2 at (152.4, 128.9)
- removed the U5 at (153.5, 138.0)
- removed the Y1 at (137.7, 132.3)
- added 1V8: 1V8, LED_SMD:LED_0805_2012Metric, F.Cu at (127.0, 149.8)
- added 3V3: 3V3, LED_SMD:LED_0805_2012Metric, F.Cu at (123.5, 149.3)
- added 5V: VBUS_LED, LED_SMD:LED_0805_2012Metric, B.Cu at (141.7, 110.5)
- added C24: 1uF, Capacitor_SMD:C_0603_1608Metric, F.Cu at (139.0, 131.9)
- added C25: 0.1uF, Capacitor_SMD:C_0603_1608Metric, F.Cu at (143.7, 138.6)
- added C26: 0.1uF, Capacitor_SMD:C_0603_1608Metric, F.Cu at (127.5, 144.1)
- added C28: 0.1uF, Capacitor_SMD:C_0603_1608Metric, F.Cu at (133.2, 148.3)
- added C29: 12pF, Capacitor_SMD:C_0603_1608Metric, F.Cu at (135.3, 130.2)
- added C30: 12pF, Capacitor_SMD:C_0603_1608Metric, F.Cu at (135.3, 136.0)
- added C31: 0.1uF, Capacitor_SMD:C_0603_1608Metric, F.Cu at (156.2, 148.2)
- added C33: 0.1uF, Capacitor_SMD:C_0603_1608Metric, F.Cu at (143.3, 150.1)
- added C35: 0.1uF, Capacitor_SMD:C_0603_1608Metric, F.Cu at (153.1, 131.8)
- added D8: 1N4448W, Diode_SMD:D_SOD-123, F.Cu at (123.7, 132.2)
- added EEPROM: EEPROM, TestPoint:TestPoint_THTPad_D1.0mm_Drill0.5mm, F.Cu at (136.5, 149.8)
- added G***: LOGO, riscv-phone:3333dpi_silk, F.Cu at (154.2, 116.8)
- added G***: LOGO, riscv-phone:3333dpi_copper, F.Cu at (154.2, 116.7)
- added G***: LOGO, riscv-phone:bird3, B.Cu at (126.1, 112.5)
- added GND: TestPoint, TestPoint:TestPoint_Pad_2.0x2.0mm, B.Cu at (152.4, 158.9)
- added INT: INT, TestPoint:TestPoint_THTPad_D1.0mm_Drill0.5mm, F.Cu at (146.4, 148.4)
- added J6: Conn_01x03, Connector_PinHeader_2.54mm:PinHeader_1x03_P2.54mm_Vertical, F.Cu at (119.4, 140.0)
- added J7: Conn_01x10, Connector_PinHeader_2.54mm:PinHeader_1x10_P2.54mm_Vertical, F.Cu at (161.8, 153.0)
- added R1: 470, Resistor_SMD:R_0603_1608Metric, F.Cu at (123.7, 153.1)
- added R14: 4.7k, Resistor_SMD:R_0603_1608Metric, F.Cu at (154.3, 144.6)
- added R15: 4.7k, Resistor_SMD:R_0603_1608Metric, F.Cu at (155.9, 143.8)
- added R16: 4.7k, Resistor_SMD:R_0603_1608Metric, F.Cu at (146.6, 154.8)
- added R18: 100k, Resistor_SMD:R_0603_1608Metric, F.Cu at (145.2, 127.4)
- added R2: 470, Resistor_SMD:R_0603_1608Metric, F.Cu at (128.5, 152.4)
- added R3: 470, Resistor_SMD:R_0603_1608Metric, B.Cu at (138.4, 110.5)
- added R4: 470, Resistor_SMD:R_0603_1608Metric, F.Cu at (126.6, 136.4)
- added R5: 1k, Resistor_SMD:R_0603_1608Metric, F.Cu at (135.3, 128.6)
- added U4: MCP23S08_SS, Package_SO:SSOP-20_5.3x7.2mm_P0.65mm, F.Cu at (152.9, 153.2)
- added U6: M95256-WDW6P, Package_SO:TSSOP-8_4.4x3mm_P0.65mm, F.Cu at (138.3, 152.7)
- added U7: IL25LP128, Package_SO:SOIJ-8_5.3x5.3mm_P1.27mm, F.Cu at (148.6, 132.9)
- added U8: 74AHC1G08, Package_TO_SOT_SMD:SOT-23-5, F.Cu at (128.0, 140.7)
- added Y2: 16 MHz, Crystal:Crystal_SMD_3225-4Pin_3.2x2.5mm, F.Cu at (135.3, 133.1)
- C10: value 12pF -> 0.1uF
- C20: value 1uF -> 0.1uF
- C22: value 0.1uF -> 1uF
- C32: value 0.1uF -> 10nF
- D4: value SLEEP_LED -> 1V8
- H4: moved to B.Cu
- J4: value Conn_01x11 -> Conn_01x04; footprint Connector_PinHeader_2.54mm:PinHeader_1x11_P2.54mm_Vertical -> Connector_PinHeader_2.54mm:PinHeader_1x04_P2.54mm_Vertical
- J5: value Conn_01x10 -> Conn_01x08; footprint Connector_PinHeader_2.54mm:PinHeader_1x10_P2.54mm_Vertical -> Connector_PinHeader_2.54mm:PinHeader_1x08_P2.54mm_Vertical
- R10, R8: value 100k -> 1k
- R12: renamed from R26; value 10k -> 12k
- R9: renamed from R24; value 12k -> 4.7k
- U5: renamed from U1; value FE310-G000 -> FE310-G002
- moved J4 56.2 mm to (161.8, 116.0), turned to 0 degrees
- moved J3 52.2 mm to (119.4, 145.8)
- moved J5 34.7 mm to (127.2, 158.5), turned to 90 degrees
- moved R10 30.8 mm to (150.2, 122.8), turned to 0 degrees
- moved R8 30.4 mm to (147.0, 122.2)
- moved C15 29.8 mm to (139.2, 111.1)
- moved C22 29.6 mm to (146.2, 139.8)
- moved C34 27.5 mm to (129.3, 144.7), turned to 90 degrees
- moved C32 27.1 mm to (124.0, 134.2), turned to 0 degrees
- moved C20 17.0 mm to (139.9, 149.2), turned to 0 degrees
- moved C21 16.3 mm to (140.3, 134.6), turned to 0 degrees
- moved C8 15.1 mm to (147.6, 117.7), turned to 90 degrees
- moved C10 15.0 mm to (145.2, 122.2), turned to 270 degrees
- moved D4 14.5 mm to (124.0, 138.2), turned to 270 degrees
- moved C27 14.1 mm to (134.4, 138.5), turned to 270 degrees
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- renumbered C90 to C1, C35 to C11, C36 to C12, C26 to C13, C30 to C14, C24 to C16, C28 to C17, C23 to C18, C27 to C19, C92 to C2, C19 to C23, C16 to C27, C93 to C3, C91 to C4, C25 to C5, C29 to C6, C31 to C7, C33 to C9, D8 to D5, D9 to D6, D2 to D7, D5 to D9, H3 to H2, H2 to H3, J7 to J1, J1 to J2, R25 to R11, R12 to R13, R7 to R17, R29 to R6, R23 to R7, U90 to U1, U91 to U2, U9 to U3, Y2 to Y1
Connections:
- C10 pad 1: Net-(C10-Pad1) -> /Program and Debug/VCORE_FT
- C15 pad 1: +1V8 -> +3V3
- C20 pad 1: /Microcontroller/PLL_AVDD -> +1V8
- C20 pad 2: /Microcontroller/PLL_AVSS -> GND
- C21 pad 1: /Microcontroller/VDD_3V3_MOFF -> +1V8
- C22 pad 1: +3V3 -> +1V8
- C27 pad 1: /Microcontroller/VDD_3V3_MOFF -> +3V3
- C32 pad 1: +3V3 -> /Microcontroller/JTAG_SRST
- C34 pad 1: /Program and Debug/VCORE_FT -> +1V8
- C8 pad 1: /Microcontroller/VDD_3V3_MOFF -> +3V3
- D4 pad 1: GND -> Net-(D4-Pad1)
- D4 pad 2: Net-(D4-Pad2) -> /Microcontroller/1V8_EN
- D7 pad 3: /RESET -> /Microcontroller/JTAG_SRST
- D9 pad 1: /RESET -> /Microcontroller/JTAG_SRST
- J4 pad 1: /Microcontroller/RESET_N_1V8 -> GND
- J4 pad 2: /Microcontroller/KEYPAD_INT -> +3V3
- J4 pad 3: /Microcontroller/RI -> GND
- J4 pad 4: /Microcontroller/LCD_CS -> +1V8
- J5 pad 1: /Microcontroller/MODEM_RST -> /Microcontroller/RI_INT
- J5 pad 2: /Microcontroller/MODEM_STATUS -> /Microcontroller/BUZZER
- J5 pad 3: /Microcontroller/BUZZER -> /Microcontroller/KEYPAD_INT
- J5 pad 4: /Microcontroller/LCD_LED_PWM -> /Microcontroller/MISO
- J5 pad 5: /Microcontroller/LCD_DC -> /Microcontroller/MOSI
- J5 pad 6: /Microcontroller/HEADPHONE_DETECT -> /Microcontroller/SCK
- J5 pad 7: /Microcontroller/MODEM_TX -> /Microcontroller/MODEM_STATUS
- J5 pad 8: /Microcontroller/MODEM_RX -> /Microcontroller/HP_DET_INT
- R10 pad 1: +3V3 -> /Program and Debug/FT_RX
- R10 pad 2: Net-(Q1-Pad6) -> GND
- R17 pad 2: /RESET -> /Microcontroller/JTAG_SRST
- R8 pad 1: +1V8 -> /Microcontroller/DBG_TO_MCU
- R8 pad 2: /Microcontroller/WAKEUP_N -> /Program and Debug/FT_UART_TX
- R9 pad 2: Net-(Q1-Pad3) -> /Microcontroller/FT_RESET
- RST1 pad 2: /RESET -> /Microcontroller/JTAG_SRST
- U3 pad 14: Net-(Q1-Pad3) -> /Microcontroller/FT_RESET
- U3 pad 22: /RESET -> /Microcontroller/JTAG_SRST
- U3 pad 39: /Microcontroller/DEBUG_RX -> /Program and Debug/FT_RX
- U5 pad 10: Net-(C10-Pad1) -> Net-(C30-Pad1)
- U5 pad 11: /Microcontroller/VDD_3V3_MOFF -> +3V3
- U5 pad 12: /Microcontroller/VDD_3V3_MOFF -> +3V3
- U5 pad 17: /Microcontroller/VDD_PAD_EN -> /Microcontroller/1V8_EN
- U5 pad 19: +1V8 -> +3V3
- U5 pad 23: +1V8 -> +3V3
- U5 pad 24: /Microcontroller/RESET_N_1V8 -> /Microcontroller/JTAG_SRST
- U5 pad 25: /Microcontroller/KEYPAD_INT -> /Microcontroller/BUZZER
- U5 pad 26: /Microcontroller/RI -> /Microcontroller/INT_CTRL_INT
- U5 pad 27: /Microcontroller/LCD_CS -> /Microcontroller/EEPROM_CS
- U5 pad 32: /Microcontroller/VDD_3V3_MOFF -> +3V3
- U5 pad 33: /Microcontroller/EEPROM_CS -> /Microcontroller/INT_CTRL_CS
- U5 pad 34: /Microcontroller/BRIDGE_CS -> /Microcontroller/LCD_CS
- U5 pad 36: /Microcontroller/DTR -> /Microcontroller/SDA
- U5 pad 37: /Microcontroller/BUZZER -> /Microcontroller/SCL
- U5 pad 38: /Microcontroller/UART0_RX -> /Microcontroller/MODEM_TO_MCU
- U5 pad 39: /Microcontroller/UART0_TX -> /Microcontroller/MCU_TO_MODEM
- U5 pad 40: /Microcontroller/MUXSEL -> /Program and Debug/FT_RX
- U5 pad 43: /Microcontroller/HEADPHONE_DETECT -> /Microcontroller/KEYPAD_INT
- U5 pad 44: /Microcontroller/BRIDGE_INT -> /Microcontroller/DTR
- U5 pad 45: /Microcontroller/BRIDGE_WAKEUP -> /Microcontroller/DBG_TO_MCU
- U5 pad 47: /Microcontroller/VDD_3V3_MOFF -> +3V3
Routing:
- net /Microcontroller/VDD_3V3_MOFF: track 195.6 -> 0.00 mm, vias 8 -> 0
- net /Microcontroller/JTAG_SRST: track 0.00 -> 114.9 mm, vias 0 -> 1
- net +1V8: track 250.4 -> 156.0 mm, vias 16 -> 15
- net /RESET: track 79.8 -> 0.00 mm, vias 7 -> 0
- net /Microcontroller/KEYPAD_INT: track 19.7 -> 92.5 mm, vias 0 -> 4
- net /Microcontroller/RI_INT: track 0.00 -> 55.3 mm, vias 0 -> 3
- net /Program and Debug/FT_RX: track 0.00 -> 40.7 mm, vias 0 -> 2
- net /Microcontroller/DEBUG_RX: track 39.3 -> 0.00 mm, vias 2 -> 0
- net /Microcontroller/RESET_N_1V8: track 49.7 -> 13.8 mm, vias 3 -> 0
- net /Microcontroller/DEBUG_TX: track 32.7 -> 0.00 mm, vias 2 -> 0
- net /Microcontroller/DBG_TO_MCU: track 0.00 -> 31.2 mm
- net /Microcontroller/INT_CTRL_INT: track 0.00 -> 30.1 mm, vias 0 -> 4
- net /Microcontroller/FT_RESET: track 16.5 -> 44.9 mm, vias 2 -> 4
- net /Microcontroller/MODEM_TO_MCU: track 0.00 -> 27.3 mm
- net +3V3: track 258.1 -> 285.3 mm, vias 12 -> 25
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Other:
- net class pwr added: clearance 0.1524, trace_width 0.2286, via_dia 0.6858, via_drill 0.3302
- board text added: "1V8 EN"
- board text added: "KP INT"
- board text added: "LCD D/C"
- board text added: "Spencer Moss"
- board text added: "rev 2.0"
- board text added: "~RST"
- board text added: "~RST 1V8"
- board text removed: "3V3 MOFF"
- board text removed: "KEY INT"
- board text removed: "LCD DC"
- board text removed: "Layout: Spencer Moss"
- board text removed: "RESET"
- board text removed: "RESET_N 1V8"
- board text removed: "rev 1.1"
